File: docs/electrical/station_revD_20261021/kicad/RoomCleaner_Station_RevD.kicad_sch (KiCad schematic)
At the start: 14 parts, among them J1 12V_IN, J2 MOTOR_NEMA17, J3 SWITCH_KW12-3, J5 ENCODER_AS5600, U1 DROK_buck_5.00V, U2 XIAO_ESP32C3, U3 A4988_carrier

Commit message: Station Rev D KiCad project: schematic (ERC 0/0), netlist matches perfboard (16 nets, PASS), placed 70x50 mm PCB (DRC: unrouted only), generator and checks
Co-Authored-By: Claude Opus 5.5 <noreply@anthropic.com>
Claude-Session: https://claude.ai/code/session_012vxDhJBdXDDzxaEvKJXH5D
Other:
- note added: "D1 1N5819, stripe (cathode) toward the XIAO. Blocks back- feed into the buck; not an over-voltage clamp."
- note added: "J1: pin 1 +12 V, pin 2 GND (perfboard X01, X03, 5.08 mm terminal or wires). 12 V comes from the supply branch; the PWR_FLAGs mark J1 as the source. C1 sits at VMOT (perfboard T02 +, T03 -)."
- note removed: "D1 1N5819, stripe (cathode) toward the XIAO. Blocks back-feed into the buck; it is not an over-voltage clamp."
- note removed: "J1 pin 1 +12 V, pin 2 GND (perfboard X01, X03; 5.08 mm terminal or wires). 12 V comes from the supply branch: the PWR_FLAGs mark the connector as the source. C1 sits at VMOT (perfboard T02 +, T03 -)."
- moved on the sheet: U2
Changed lines of the file:
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@@
     )
   )
-  (text "J1 pin 1 +12 V, pin 2 GND (perfboard X01, X03; 5.08 mm terminal or wires).\n12 V comes from the supply branch: the PWR_FLAGs mark the connector as the source.\nC1 sits at VMOT (perfboard T02 +, T03 -)." (at 15.24 73.66 0)
+  (text "J1: pin 1 +12 V, pin 2 GND (perfboard X01, X03,\n5.08 mm terminal or wires).  12 V comes from the\nsupply branch; the PWR_FLAGs mark J1 as the source.\nC1 sits at VMOT (perfboard T02 +, T03 -)." (at 15.24 73.66 0)
     (effects (font (size 1.27 1.27)) (justify left top))
   )
@@
     )
   )
-  (text "U1 EN is unconnected (as soldered).  Select 5 V with the module's 5V pad;\nset and check 5.00 V BEFORE connecting loads.  Non-isolated: IN- = OUT-." (at 92.71 76.2 0)
-    (effects (font (size 1.27 1.27)) (justify left top))
-  )
-  (text "D1 1N5819, stripe (cathode) toward the XIAO.\nBlocks back-feed into the buck;\nit is not an over-voltage clamp." (at 137.16 58.42 0)
-    (effects (font (size 1.27 1.27)) (justify left top))
-  )
-  (text "JP1: OPEN while USB is plugged in.\nCLOSED standalone from 12 V.\nChange only with all power off." (at 171.45 58.42 0)
-    (effects (font (size 1.27 1.27)) (justify left top))
-  )
-  (text "PWR_FLAG on +5V: 5 V comes from USB VBUS or from the buck through D1 + JP1\n(never both at once)." (at 137.16 70 0)
+  (text "U1 EN is unconnected (as soldered).  Select 5 V with the\nmodule's 5V pad; set and check 5.00 V BEFORE connecting\nloads.  Non-isolated: IN- = OUT-." (at 92.71 76.2 0)
+    (effects (font (size 1.27 1.27)) (justify left top))
+  )
+  (text "D1 1N5819, stripe (cathode)\ntoward the XIAO. Blocks back-\nfeed into the buck; not an\nover-voltage clamp." (at 137.16 62.23 0)
+    (effects (font (size 1.27 1.27)) (justify left top))
+  )
+  (text "JP1: OPEN while USB is plugged in.\nCLOSED standalone from 12 V.\nChange only with all power off." (at 172.72 62.23 0)
+    (effects (font (size 1.27 1.27)) (justify left top))
+  )
+  (text "PWR_FLAG on +5V: 5 V comes from USB VBUS or from\nthe buck through D1 + JP1 (never both at once)." (at 172.72 76.2 0)
     (effects (font (size 1.27 1.27)) (justify left top))
   )
@@
   (symbol (lib_id "RoomCleaner:XIAO_ESP32C3") (at 63.5 142.24 0) (unit 1)
     (in_bom yes) (on_board yes) (dnp no)
-    (property "Reference" "U2" (at 57.15 111.76 0)
+    (property "Reference" "U2" (at 57.15 107.95 0)
       (effects (font (size 1.27 1.27)) (justify left))
     )
-    (property "Value" "XIAO_ESP32C3" (at 57.15 114.3 0)
+    (property "Value" "XIAO_ESP32C3" (at 57.15 110.49 0)
       (effects (font (size 1.27 1.27)) (justify left))
     )
@@
     (effects (font (size 1.27 1.27)) (justify right bottom))
   )
-  (text "J2 MOTOR (X05-X08): pins 1-4 =\n2B 2A 1A 1B.  1A/1B = coil 1,\n2A/2B = coil 2.\nNever plug / unplug the motor\nwith power on." (at 270.51 157.48 0)
+  (text "J2 MOTOR (X05-X08): pins 1-4 =\n2B 2A 1A 1B.  1A/1B = coil 1,\n2A/2B = coil 2.\nNever plug / unplug the motor\nwith power on." (at 261.62 157.48 0)
     (effects (font (size 1.27 1.27)) (justify left top))
   )
@@
     (effects (font (size 1.27 1.27)) (justify left top))
   )
-  (rectangle (start 170.18 196) (end 297.18 252)
+  (rectangle (start 170.18 196) (end 297.18 247)
     (stroke (width 0.254) (type default))
     (fill (type none))
@@
     (effects (font (size 1.27 1.27)) (justify left top))
   )
-  (text "MICROSTEP (MS1/MS2/MS3): all three tied LOW (GND) = FULL STEP -> config `microsteps` = 1\n(config/robot.example.json). If they are moved to +3V3 (1/16 step) set `microsteps` = 16 for\nthat station before the first run. Hardware and config MUST match: mismatch = wrong lengths." (at 172.72 219 0)
-    (effects (font (size 1.27 1.27)) (justify left top))
-  )
-  (text "DO NOT RAISE VDD TO 5 V. A4988 VDD, RESET, SLEEP = 3.3 V from the XIAO 3V3 pin; the ESP32-C3\nGPIOs (STEP, DIR, EN) are not 5 V tolerant.  Pull-ups to 3.3 V only." (at 172.72 232 0)
-    (effects (font (size 1.27 1.27)) (justify left top))
-  )
-  (text "FUSING IS AT THE SUPPLY END: branch fuses F1-F4 (rating TBD) and F0 7.5 A (existing, recorded,\nnot approved) sit before the long cables. No fuse, reverse-polarity or over-voltage protection\non this board. Rev D TP0-TP4 are not parts on the perfboard: probe the module pins / holes." (at 172.72 240 0)
+  (text "MICROSTEP (MS1/MS2/MS3): all three tied LOW (GND) = FULL STEP -> config `microsteps` = 1\n(config/robot.example.json). If they are moved to +3V3 (1/16 step) set `microsteps` = 16 for\nthat station before the first run. Hardware and config MUST match: mismatch = wrong lengths." (at 172.72 214 0)
+    (effects (font (size 1.27 1.27)) (justify left top))
+  )
+  (text "DO NOT RAISE VDD TO 5 V. A4988 VDD, RESET, SLEEP = 3.3 V from the XIAO 3V3 pin; the ESP32-C3\nGPIOs (STEP, DIR, EN) are not 5 V tolerant.  Pull-ups to 3.3 V only." (at 172.72 224 0)
+    (effects (font (size 1.27 1.27)) (justify left top))
+  )
+  (text "FUSING IS AT THE SUPPLY END: branch fuses F1-F4 (rating TBD) and F0 7.5 A (existing, recorded,\nnot approved) sit before the long cables. No fuse, reverse-polarity or over-voltage protection\non this board. Rev D TP0-TP4 are not parts on the perfboard: probe the module pins / holes." (at 172.72 232 0)
     (effects (font (size 1.27 1.27)) (justify left top))
   )
@@
     (effects (font (size 1.27 1.27)) (justify left top))
   )
-  (text "USB / EXTERNAL POWER" (at 304.8 76.2 0)
+  (text "USB / EXTERNAL POWER" (at 304.8 62 0)
     (effects (font (size 1.8 1.8) bold) (justify left top))
   )
-  (text "USB plugged in: JP1 OPEN.  Standalone from 12 V: USB unplugged,\nJP1 CLOSED.  Never USB + 12 V with JP1 closed (two sources meet\non VBUS).  Change JP1 only with all power off." (at 304.8 81.28 0)
-    (effects (font (size 1.27 1.27)) (justify left top))
-  )
-  (text "PERFBOARD HOLE MAP (generated, component side, A01 top-left)" (at 304.8 94 0)
+  (text "USB plugged in: JP1 OPEN.  Standalone from 12 V: USB unplugged,\nJP1 CLOSED.  Never USB + 12 V with JP1 closed (two sources meet\non VBUS).  Change JP1 only with all power off." (at 304.8 67.1 0)
+    (effects (font (size 1.27 1.27)) (justify left top))
+  )
+  (text "PERFBOARD HOLE MAP (generated, component side, A01 top-left)" (at 304.8 82 0)
     (effects (font (size 1.8 1.8) bold) (justify left top))
   )
-  (text "J1: 1=X01  2=X03\nJ2: 1=X05  2=X06  3=X07  4=X08\nJ5: 1=C17  2=D17  3=E17  4=F17\nJ3: 1=H17  2=I17\nJP1: 1=S11  2=R11\nC1: 1=T02  2=T03\nD1: 1=T11  2=X11\nU1: 1=X15  2=W15  3=V15  4=U15  5=T15\nR1: E13 - E10\nR2: C10 - C11\nR3: D10 - D11\nR4: H13 - H16\nU2: B03..H03 (5V..D7) and B09..H09 (D0..D6)\nU3: L03..L10 (pads 9..16) and Q03..Q10 (pads 8..1)\n\nPin 1 = first hole listed.  U1 EN (T15) and XIAO D0, D6, D7,\nD8, D9 are unconnected on the board (no-connect flags)." (at 304.8 99.06 0)
-    (effects (font (size 1.27 1.27)) (justify left top))
-  )
-  (text "DIFFERENCES FROM THE REV D SCHEMATIC (perfboard wins)" (at 304.8 140 0)
+  (text "J1: 1=X01  2=X03\nJ2: 1=X05  2=X06  3=X07  4=X08\nJ5: 1=C17  2=D17  3=E17  4=F17\nJ3: 1=H17  2=I17\nJP1: 1=S11  2=R11\nC1: 1=T02  2=T03\nD1: 1=T11  2=X11\nU1: 1=X15  2=W15  3=V15  4=U15  5=T15\nR1: E13 - E10\nR2: C10 - C11\nR3: D10 - D11\nR4: H13 - H16\nU2: B03..H03 (5V..D7) and B09..H09 (D0..D6)\nU3: L03..L10 (pads 9..16) and Q03..Q10 (pads 8..1)\n\nPin 1 = first hole listed.  U1 EN (T15) and XIAO D0, D6, D7,\nD8, D9 are unconnected on the board (no-connect flags)." (at 304.8 87.1 0)
+    (effects (font (size 1.27 1.27)) (justify left top))
+  )
+  (text "DIFFERENCES FROM THE REV D SCHEMATIC (perfboard wins)" (at 304.8 128 0)
     (effects (font (size 1.8 1.8) bold) (justify left top))
   )
-  (text "Current limit: Rev D sheet 3 / README show 1.35 A, Vref 1.08 V (D29).\n  This sheet follows D30: Vref 0.85 V, about 1.06 A.\nEncoder: Rev D sheet 3 draws DIR to GND and OUT open at the encoder.\n  The board has a 4-pin J5 only (3V3, GND, SDA, SCL), so those two\n  are on the encoder board, not on the perfboard.\nTest points TP0-TP4 of Rev D are not parts on the perfboard.\nGrounds: Rev D shows one GND; the board has two A4988 GND pads (pad 7\n  motor return, pad 1 logic) tied by wire S03-O11 = one GND net here.\nPackages as built: R2/R3 stand upright (2.54 mm), R1/R4 lie (7.62 mm);\n  J1 is a 5.08 mm terminal pitch (2.54 mm header otherwise).\nNet names: perfboard 3V3 / 5V / 12V are the +3V3 / +5V / +12V power\n  symbols; 5VB = buck OUT+ / D1 anode, 5VD = D1 cathode / JP1." (at 304.8 145 0)
-    (effects (font (size 1.27 1.27)) (justify left top))
-  )
+  (text "Current limit: Rev D sheet 3 / README show 1.35 A, Vref 1.08 V (D29).\n  This sheet follows D30: Vref 0.85 V, about 1.06 A.\nEncoder: Rev D sheet 3 draws DIR to GND and OUT open at the encoder.\n  The board has a 4-pin J5 only (3V3, GND, SDA, SCL), so those two\n  are on the encoder board, not on the perfboard.\nTest points TP0-TP4 of Rev D are not parts on the perfboard.\nGrounds: Rev D shows one GND; the board has two A4988 GND pads (pad 7\n  motor return, pad 1 logic) tied by wire S03-O11 = one GND net here.\nPackages as built: R2/R3 stand upright (2.54 mm), R1/R4 lie (7.62 mm);\n  J1 is a 5.08 mm terminal pitch (2.54 mm header otherwise).\nNet names: perfboard 3V3 / 5V / 12V are the +3V3 / +5V / +12V power\n  symbols; 5VB = buck OUT+ / D1 anode, 5VD = D1 cathode / JP1." (at 304.8 133.1 0)
+    (effects (font (size 1.27 1.27)) (justify left top))
+  )
